Commit message: xarm implementation, working but still the grasp feels not natural

File: grasp_generation/assets/urdf/xarm7_dexhand/xarm7_allegro_right.urdf (robot description, URDF)
Before this commit: robot xarm7, 32 links, 31 joints
Links:
- link base_link: geometry collision box size=0.0414 0.0538 0.0428; collision box size=0.0414 0.0720 0.013
- link link_0.0: geometry collision box size=0.0196 0.0275 0.0164; visual mesh filename=allegro/meshes/visual/link_0.glb
- link link_1.0: geometry collision box size=0.0196 0.0275 0.054; visual mesh filename=allegro/meshes/visual/link_1.glb
- link link_10.0: geometry collision box size=0.0196 0.0275 0.0384; visual mesh filename=allegro/meshes/visual/link_2.glb
- link link_11.0: geometry collision box size=0.0196 0.0269 0.022; visual mesh filename=allegro/meshes/visual/link_3.glb
- link link_11.0_tip: geometry collision mesh filename=allegro/meshes/collision/link_tip.obj; visual mesh filename=allegro/meshes/visual/link_tip.glb
- link link_12.0: geometry collision box size=0.0358 0.034 0.0455; visual mesh filename=allegro/meshes/visual/link_12_right.glb
- link link_13.0: geometry collision box size=0.0196 0.0275 0.0177; visual mesh filename=allegro/meshes/visual/link_13.glb
- link link_14.0: geometry collision box size=0.0196 0.0275 0.0514; visual mesh filename=allegro/meshes/visual/link_14.glb
- link link_15.0: geometry collision box size=0.0196 0.0269 0.04; visual mesh filename=allegro/meshes/visual/link_15.glb
- link link_15.0_tip: geometry collision mesh filename=allegro/meshes/collision/link_tip.obj; visual mesh filename=allegro/meshes/visual/link_tip.glb
- link link_2.0: geometry collision box size=0.0196 0.0275 0.0384; visual mesh filename=allegro/meshes/visual/link_2.glb
- link link_3.0: geometry collision box size=0.0196 0.0269 0.022; visual mesh filename=allegro/meshes/visual/link_3.glb
- link link_3.0_tip: geometry collision mesh filename=allegro/meshes/collision/link_tip.obj; visual mesh filename=allegro/meshes/visual/link_tip.glb
- link link_4.0: geometry collision box size=0.0196 0.0275 0.0164; visual mesh filename=allegro/meshes/visual/link_0.glb
- link link_5.0: geometry collision box size=0.0196 0.0275 0.054; visual mesh filename=allegro/meshes/visual/link_1.glb
- link link_6.0: geometry collision box size=0.0196 0.0275 0.0384; visual mesh filename=allegro/meshes/visual/link_2.glb
- link link_7.0: geometry collision box size=0.0196 0.0269 0.022; visual mesh filename=allegro/meshes/visual/link_3.glb
- link link_7.0_tip: geometry collision mesh filename=allegro/meshes/collision/link_tip.obj; visual mesh filename=allegro/meshes/visual/link_tip.glb
- link link_8.0: geometry collision box size=0.0196 0.0275 0.0164; visual mesh filename=allegro/meshes/visual/link_0.glb
- link link_9.0: geometry collision box size=0.0196 0.0275 0.054; visual mesh filename=allegro/meshes/visual/link_1.glb
- link part_studio_link: geometry collision mesh filename=hand_mount/meshes/collision/mount_v4.stl scale=0.001 0.001 0.001; visual mesh filename=hand_mount/meshes/visual/mount_v4.stl scale=0.001 0.001 0.001
Joints:
- removed joint joint1
- removed joint joint2
- removed joint joint3
- removed joint joint4
- removed joint joint5
- removed joint joint6
- removed joint joint7
- added joint xarm7_joint1: type revolute, parent link_base, child link1, origin xyz=0 0 0.267 rpy=0 0 0, axis 0 0 1, limit lower=-6.28318530718 upper=6.28318530718 effort=50 velocity=3.14
- added joint xarm7_joint2: type revolute, parent link1, child link2, origin xyz=0 0 0 rpy=-1.5708 0 0, axis 0 0 1, limit lower=-2.059 upper=2.0944 effort=50 velocity=3.14
- added joint xarm7_joint3: type revolute, parent link2, child link3, origin xyz=0 -0.293 0 rpy=1.5708 0 0, axis 0 0 1, limit lower=-6.28318530718 upper=6.28318530718 effort=30 velocity=3.14
- added joint xarm7_joint4: type revolute, parent link3, child link4, origin xyz=0.0525 0 0 rpy=1.5708 0 0, axis 0 0 1, limit lower=-0.19198 upper=3.927 effort=30 velocity=3.14
- added joint xarm7_joint5: type revolute, parent link4, child link5, origin xyz=0.0775 -0.3425 0 rpy=1.5708 0 0, axis 0 0 1, limit lower=-6.28318530718 upper=6.28318530718 effort=30 velocity=3.14
- added joint xarm7_joint6: type revolute, parent link5, child link6, origin xyz=0 0 0 rpy=1.5708 0 0, axis 0 0 1, limit lower=-1.69297 upper=3.14159265359 effort=20 velocity=3.14
- added joint xarm7_joint7: type revolute, parent link6, child link7, origin xyz=0.076 0.097 0 rpy=-1.5708 0 0, axis 0 0 1, limit lower=-6.28318530718 upper=6.28318530718 effort=20 velocity=3.14

File: grasp_generation/assets/urdf/xarm7_dexhand/xarm7_leap_right.urdf (robot description, URDF)
Before this commit: robot xarm7, 25 links, 24 joints
Links:
- removed link dip
- removed link fingertip
- removed link mcp_joint
- removed link palm_lower
- removed link pip
- added link dip_1, mass 0.037; collision mesh filename=leap_hand/dip.stl; visual mesh filename=leap_hand/dip.stl
- added link fingertip_1, mass 0.016; collision mesh filename=leap_hand/fingertip.stl; visual mesh filename=leap_hand/fingertip.stl
- added link mcp_joint_1, mass 0.044; collision mesh filename=leap_hand/mcp_joint.stl; visual mesh filename=leap_hand/mcp_joint.stl
- added link palm_link, mass 0.237; collision mesh filename=leap_hand/palm_lower.stl; visual mesh filename=leap_hand/palm_lower.stl
- added link pip_1, mass 0.032; collision mesh filename=leap_hand/pip.stl; visual mesh filename=leap_hand/pip.stl
- link dip_2: geometry collision mesh filename=leap_hand/dip.stl; visual mesh filename=leap_hand/dip.stl
- link dip_3: geometry collision mesh filename=leap_hand/dip.stl; visual mesh filename=leap_hand/dip.stl
- link fingertip_2: geometry collision mesh filename=leap_hand/fingertip.stl; visual mesh filename=leap_hand/fingertip.stl
- link fingertip_3: geometry collision mesh filename=leap_hand/fingertip.stl; visual mesh filename=leap_hand/fingertip.stl
- link mcp_joint_2: geometry collision mesh filename=leap_hand/mcp_joint.stl; visual mesh filename=leap_hand/mcp_joint.stl
- link mcp_joint_3: geometry collision mesh filename=leap_hand/mcp_joint.stl; visual mesh filename=leap_hand/mcp_joint.stl
- link pip_2: geometry collision mesh filename=leap_hand/pip.stl; visual mesh filename=leap_hand/pip.stl
- link pip_3: geometry collision mesh filename=leap_hand/pip.stl; visual mesh filename=leap_hand/pip.stl
- link pip_4: geometry collision mesh filename=leap_hand/pip.stl; visual mesh filename=leap_hand/pip.stl
- link thumb_dip: geometry collision mesh filename=leap_hand/thumb_dip.stl; visual mesh filename=leap_hand/thumb_dip.stl
- link thumb_fingertip: geometry collision mesh filename=leap_hand/thumb_fingertip.stl; visual mesh filename=leap_hand/thumb_fingertip.stl
- link thumb_pip: geometry collision mesh filename=leap_hand/thumb_pip.stl; visual mesh filename=leap_hand/thumb_pip.stl
Joints:
- removed joint joint1
- removed joint joint2
- removed joint joint3
- removed joint joint4
- removed joint joint5
- removed joint joint6
- removed joint joint7
- removed joint joint_0
- removed joint joint_1
- removed joint joint_10
- removed joint joint_11
- removed joint joint_12
- removed joint joint_13
- removed joint joint_14
- removed joint joint_15
- removed joint joint_2
- removed joint joint_3
- removed joint joint_4
- removed joint joint_5
- removed joint joint_6
- removed joint joint_7
- removed joint joint_8
- removed joint joint_9
- added joint leap_joint0: type revolute, parent mcp_joint_1, child pip_1, origin xyz=-0.012200000000000007713 0.038099999999999994982 0.014500000000000000736 rpy=-1.570796326794896558 -1.0065212660796336576e-15 1.5707963267948943376, axis 0 0 -1, limit lower=-1.047 upper=1.047 effort=0.95 velocity=8.48
- added joint leap_joint1: type revolute, parent palm_link, child mcp_joint_1, origin xyz=-0.0070952496528625457958 0.023057756134899472233 -0.01872240357846021927 rpy=1.5707963267948950037 1.5707963267948945596 0, axis 0 0 -1, limit lower=-0.314 upper=2.23 effort=0.95 velocity=8.48
- added joint leap_joint10: type revolute, parent pip_3, child dip_3, origin xyz=0.014999999999999971689 0.014299999999999951639 -0.012999999999999959505 rpy=1.5707963267948958919 -1.570796326794896336 0, axis 0 0 -1, limit lower=-0.506 upper=1.885 effort=0.95 velocity=8.48
- added joint leap_joint11: type revolute, parent dip_3, child fingertip_3, origin xyz=9.7144514654701197287e-17 -0.036099999999999868305 0.00020000000000007511769 rpy=4.5935029425113685044e-17 -2.8730071914463799514e-16 1.5565411607615035382e-32, axis 0 0 -1, limit lower=-0.366 upper=2.042 effort=0.95 velocity=8.48
- added joint leap_joint12: type revolute, parent palm_link, child pip_4, origin xyz=-0.069395249652862533996 -0.0012422438651005258004 -0.021622403578460215601 rpy=-8.2381766464939424156e-17 1.5707963267948956698 0, axis 0 0 -1, limit lower=-0.349 upper=2.094 effort=0.95 velocity=8.48
- added joint leap_joint13: type revolute, parent pip_4, child thumb_pip, origin xyz=-2.7755575615628913511e-17 0.014300000000000005415 -0.013000000000000011546 rpy=1.5707963267948958919 -1.570796326794896336 0, axis 0 0 -1, limit lower=-0.47 upper=2.443 effort=0.95 velocity=8.48
- added joint leap_joint14: type revolute, parent thumb_pip, child thumb_dip, origin xyz=0 0.014499999999999966041 -0.017000000000000053263 rpy=-1.570796326794896558 1.6050198443300131245e-46 -1.9721522630516624601e-31, axis 0 0 -1, limit lower=-1.20 upper=1.90 effort=0.95 velocity=8.48
- added joint leap_joint15: type revolute, parent thumb_dip, child thumb_fingertip, origin xyz=-1.249000902703301108e-16 0.046599999999999863753 0.00019999999999997710581 rpy=1.5063958491491781023e-44 5.4234187233935260503e-31 3.141592653589793116, axis 0 0 -1, limit lower=-1.34 upper=1.88 effort=0.95 velocity=8.48
- added joint leap_joint2: type revolute, parent pip_1, child dip_1, origin xyz=0.01499999999999996822 0.014299999999999904801 -0.012999999999999824196 rpy=1.5707963267948958919 -1.570796326794896336 0, axis 0 0 -1, limit lower=-0.506 upper=1.885 effort=0.95 velocity=8.48
- added joint leap_joint3: type revolute, parent dip_1, child fingertip_1, origin xyz=-4.0880582495572692636e-09 -0.036100004210367367397 0.00020000000000007858714 rpy=4.5935029425113685044e-17 -2.8730071914463794583e-16 4.4395481053923607589e-32, axis 0 0 -1, limit lower=-0.366 upper=2.042 effort=0.95 velocity=8.48
- added joint leap_joint4: type revolute, parent mcp_joint_2, child pip_2, origin xyz=-0.012200000000000019856 0.038099999999999981104 0.01450000000000000594 rpy=-1.570796326794896558 -1.0065212760057939085e-15 1.5707963267948943376, axis 0 0 -1, limit lower=-1.047 upper=1.047 effort=0.95 velocity=8.48
- added joint leap_joint5: type revolute, parent palm_link, child mcp_joint_2, origin xyz=-0.0070952496528625388569 -0.022392243865100525113 -0.018722403578460229678 rpy=1.570796326794896558 1.570796326794896558 0, axis 0 0 -1, limit lower=-0.314 upper=2.23 effort=0.95 velocity=8.48
- added joint leap_joint6: type revolute, parent pip_2, child dip_2, origin xyz=0.014999999999999975159 0.014300000000000000211 -0.013000000000000018485 rpy=1.5707963267948958919 -1.570796326794896336 0, axis 0 0 -1, limit lower=-0.506 upper=1.885 effort=0.95 velocity=8.48
- added joint leap_joint7: type revolute, parent dip_2, child fingertip_2, origin xyz=1.0061396160665481148e-16 -0.036099999999999854428 0.00020000000000007858714 rpy=4.5935029425113654229e-17 -2.8730071914463794583e-16 1.4408183216511868558e-31, axis 0 0 -1, limit lower=-0.366 upper=2.042 effort=0.95 velocity=8.48
- added joint leap_joint8: type revolute, parent mcp_joint_3, child pip_3, origin xyz=-0.012200000000000004244 0.038100000000000001921 0.014499999999999999001 rpy=-1.570796326794896558 -1.0065212660796360242e-15 1.5707963267948943376, axis 0 0 -1, limit lower=-1.047 upper=1.047 effort=0.95 velocity=8.48
- added joint leap_joint9: type revolute, parent palm_link, child mcp_joint_3, origin xyz=-0.0070952454426398371343 -0.067842243865100515521 -0.018722407666402932774 rpy=1.5707963267948950037 1.5707963267948945596 0, axis 0 0 -1, limit lower=-0.314 upper=2.23 effort=0.95 velocity=8.48
- added joint xarm7_joint1: type revolute, parent link_base, child link1, origin xyz=0 0 0.267 rpy=0 0 0, axis 0 0 1, limit lower=-6.28318530718 upper=6.28318530718 effort=50 velocity=3.14
- added joint xarm7_joint2: type revolute, parent link1, child link2, origin xyz=0 0 0 rpy=-1.5708 0 0, axis 0 0 1, limit lower=-2.059 upper=2.0944 effort=50 velocity=3.14
- added joint xarm7_joint3: type revolute, parent link2, child link3, origin xyz=0 -0.293 0 rpy=1.5708 0 0, axis 0 0 1, limit lower=-6.28318530718 upper=6.28318530718 effort=30 velocity=3.14
- added joint xarm7_joint4: type revolute, parent link3, child link4, origin xyz=0.0525 0 0 rpy=1.5708 0 0, axis 0 0 1, limit lower=-0.19198 upper=3.927 effort=30 velocity=3.14
- added joint xarm7_joint5: type revolute, parent link4, child link5, origin xyz=0.0775 -0.3425 0 rpy=1.5708 0 0, axis 0 0 1, limit lower=-6.28318530718 upper=6.28318530718 effort=30 velocity=3.14
- added joint xarm7_joint6: type revolute, parent link5, child link6, origin xyz=0 0 0 rpy=1.5708 0 0, axis 0 0 1, limit lower=-1.69297 upper=3.14159265359 effort=20 velocity=3.14
- added joint xarm7_joint7: type revolute, parent link6, child link7, origin xyz=0.076 0.097 0 rpy=-1.5708 0 0, axis 0 0 1, limit lower=-6.28318530718 upper=6.28318530718 effort=20 velocity=3.14
- joint part_studio_joint: child palm_lower -> palm_link
